Commit message: Automated update by GitHub Action

File: urdf/robot.urdf (robot description, URDF)
Before this commit: robot robot, 2 links, 1 joints
Links:
- added link camera_link, mass 1e-9
Joints:
- added joint camera_link_frame: type fixed, parent part_1, child camera_link, origin xyz=-8.05759e-05 -0.0777769 0.00836815 rpy=-0.139625 3.04604e-07 -4.28088e-08, axis 0 0 0
